Commit message: feat(robot): 新增深度相机（depth_camera），0.50 m 支架 + 110° 垂直视场
语义导航需要物体的三维位置。现有传感器不足以支撑测深：
- 双目基线仅 0.05 m、hFOV 120°（f≈185 px），1 m 处视差 9 px、2 m 处 4.6 px，
  能出图但不能测深；
- ToF 只有 16x8=128 点，4 m 处射线间距 0.52 m，0.9 m 宽的冰箱不足 2 列。

实测（本机 4 vCPU / 无 GPU / llvmpipe）：
- ogre1 渲染引擎支持 depth_camera，无需换 ogre2
- 输出 32FC1，有效像素 96%，K 与配置一致
- 相机开销可忽略：开相机 realtime_factor 0.5286 vs 不开 0.5131

安装高度与视场是实测推导的结果，不是拍脑袋定的：
车体只有 6.65 cm 高，前向传感器原装在 4.58 cm。冰箱高 1.78 m，
1.5 m 处顶端仰角 atan((1.78-0.046)/1.5)=49.3°，而原 vFoV 约 72°(±36)，
视野框不住 → 近距离看不到高物体。
方案：抬高到 0.50 m（仰角降到 40.5°）+ 垂直视场加到 110°（±55°）。
gz 的 camera 只有 horizontal_fov，垂直视场由宽高比决定，故 640x914。
实测 1.5 m 处可见 0.0~2.64 m，完整覆盖冰箱并有余量。

改动：
- params.xacro：新增 depth_camera_* 参数组 + 推导说明
- robot.urdf.xacro：depth_camera 宏（link + optical frame，rpy REP-103）
- plugins.xacro：enable_depth 开关（默认 false）+ 传感器定义
- gz_bridge.yaml：桥接 depth_camera/depth 与 depth_camera/camera_info
- sim.launch.py：enable_depth 透传

注意 gz 话题名（实测，勿按 RGB 的 /image 后缀类推）：
图在 depth_camera、info 在 /camera_info、点云在 depth_camera/points。

enable_depth 默认 false，基线 nav（SR 100% / SPL 0.988）不受影响。

File: src/semnav_robot/urdf/params.xacro (robot description, xacro)
@@ -123,4 +123,37 @@
   <xacro:property name="camera_size" value="0.010"/>               <!-- visual cube edge (m) -->
   <xacro:property name="camera_mass" value="0.005"/>               <!-- kg, negligible -->
+  <!-- ****************** DEPTH CAMERA ****************** -->
+  <!-- 语义导航的深度来源。gz 原生 depth_camera（R_FLOAT32 单通道 -> 32FC1），
+       不是双目视差。装车体前表面、中高（与 tof_front 同位置）。
+       为什么必须补这一路（两条实测依据，不是猜测）：
+       1) 双目 baseline 只有 0.05 m。120 deg hFOV、640 px 下 f 约 185 px，
+          1 m 处视差仅 9 px、2 m 处 4.6 px，低于可靠亚像素范围
+          —— 本质是「能出图、不能测深」。
+       2) 前向 ToF 是 16x8 = 128 点。4 m 处水平射线间距 0.52 m，
+          冰箱宽 0.9 m 只覆盖不到 2 列，物体级定位过稀。
+       90 deg 水平 FoV 覆盖正前方主视区；640x480 与原双目一致，
+       bbox 逻辑可复用。10 Hz：深度只用于定位，不需要高频。
+       量程 0.05-5.0 m —— 物体定位都在 3 m 内。 -->
+  <xacro:property name="depth_camera_mount_height" value="0.50"/>
+  <!-- 安装高度 0.50 m，垂直 FoV 110 deg。
+       为什么是这个组合（实测推导，不是拍的）：
+       车体只有 6.65 cm 高，前向传感器原装在 4.58 cm。冰箱（official_refrigerator）
+       高 1.78 m，在 1.5 m 距离处顶端仰角 = atan((1.78-0.046)/1.5) = 49.3 deg。
+       原 vFoV 仅约 72 deg（±36），顶端落在视野外 —— 近距离根本看不到高物体。
+       要覆盖它需同时满足：
+         1) 抬高，减小仰角：0.50 m 时仰角 atan(1.28/1.5) = 40.5 deg
+         2) 加大垂直 FoV 到 110 deg（±55 deg）
+       代价：车体上多一根 0.5 m 支架，外观不再像纯扫地机器人。
+       换来的是停靠观察时能完整看到目标物，这对阶段四的「重新观察确认」是必需的。 -->
+  <xacro:property name="depth_camera_width" value="640"/>
+  <xacro:property name="depth_camera_height" value="914"/>
+  <xacro:property name="depth_camera_hfov_deg" value="90.0"/>
+  <xacro:property name="depth_camera_near" value="0.05"/>          <!-- m -->
+  <xacro:property name="depth_camera_far" value="5.0"/>            <!-- m -->
+  <xacro:property name="depth_camera_update_rate" value="10"/>     <!-- Hz -->
+  <xacro:property name="depth_camera_x" value="${base_diameter/2}"/> <!-- 前表面 -->
+  <xacro:property name="depth_camera_z" value="${depth_camera_mount_height}"/>
+  <xacro:property name="depth_camera_size" value="0.010"/>         <!-- visual cube edge -->
+  <xacro:property name="depth_camera_mass" value="0.005"/>         <!-- kg -->
   <!-- ****************** IMU ****************** -->
   <!-- 6-axis IMU (gyro + accelerometer) near the body center. Orientation is

File: src/semnav_robot/urdf/plugins.xacro (robot description, xacro)
@@ -29,4 +29,5 @@
   <xacro:arg name="enable_tof" default="true"/>
   <xacro:arg name="enable_cameras" default="false"/>
+  <xacro:arg name="enable_depth" default="false"/>
   <xacro:arg name="enable_imu" default="true"/>
   <gazebo>
@@ -277,4 +278,32 @@
     <xacro:camera_plugin side="right"/>
   </xacro:if>
+  <!-- Depth camera (gz depth_camera -> ROS 32FC1 Image + CameraInfo).
+       gz 原生深度，非双目视差。参数见 urdf/params.xacro。
+       桥接见 config/gz_bridge.yaml 的 depth_camera/depth + camera_info 两条。 -->
+  <xacro:if value="${'$(arg enable_depth)' == 'true'}">
+  <gazebo reference="depth_camera_link">
+    <sensor name="depth_camera" type="depth_camera">
+      <pose relative_to="depth_camera_link">0 0 0 0 0 0</pose>
+      <update_rate>${depth_camera_update_rate}</update_rate>
+      <topic>depth_camera</topic>
+      <gz_frame_id>depth_camera_optical_frame</gz_frame_id>
+      <camera>
+        <horizontal_fov>${depth_camera_hfov_deg * DEG2RAD}</horizontal_fov>
+        <image>
+          <width>${depth_camera_width}</width>
+          <height>${depth_camera_height}</height>
+          <format>R_FLOAT32</format>
+        </image>
+        <clip>
+          <near>${depth_camera_near}</near>
+          <far>${depth_camera_far}</far>
+        </clip>
+        <optical_frame_id>depth_camera_optical_frame</optical_frame_id>
+      </camera>
+      <always_on>1</always_on>
+      <visualize>false</visualize>
+    </sensor>
+  </gazebo>
+  </xacro:if>
   <!-- IMU: 6-axis (gyro + accelerometer) at imu_link, near the body center. gz
        publishes gz.msgs.IMU on <topic>, bridged to sensor_msgs/Imu. Orientation

File: src/semnav_robot/urdf/robot.urdf.xacro (robot description, xacro)
@@ -107,4 +107,30 @@
     <link name="camera_${side}_optical_frame"/>
   </xacro:macro>
+  <!-- 深度相机 link + REP-103 光学坐标系（x 右、y 下、z 前）。
+       位置与 tof_front 一致（车体前表面、中高）。gz 传感器在 plugins.xacro。 -->
+  <xacro:macro name="depth_camera">
+    <joint name="depth_camera_joint" type="fixed">
+      <parent link="base_link"/>
+      <child link="depth_camera_link"/>
+      <origin xyz="${depth_camera_x} 0 ${depth_camera_z}" rpy="0 0 0"/>
+    </joint>
+    <link name="depth_camera_link">
+      <visual>
+        <origin xyz="0 0 0" rpy="0 0 0"/>
+        <geometry>
+          <box size="${depth_camera_size} ${2*depth_camera_size} ${depth_camera_size}"/>
+        </geometry>
+        <material name="dark"/>
+      </visual>
+      <xacro:solid_box_inertia m="${depth_camera_mass}"
+        x="${depth_camera_size}" y="${2*depth_camera_size}" z="${depth_camera_size}"/>
+    </link>
+    <joint name="depth_camera_optical_joint" type="fixed">
+      <parent link="depth_camera_link"/>
+      <child link="depth_camera_optical_frame"/>
+      <origin xyz="0 0 0" rpy="${-pi/2} 0 ${-pi/2}"/>
+    </joint>
+    <link name="depth_camera_optical_frame"/>
+  </xacro:macro>
   <link name="base_footprint"/>
   <joint name="base_joint" type="fixed">
@@ -237,4 +263,6 @@
   <xacro:stereo_camera side="left" side_sign="1"/>
   <xacro:stereo_camera side="right" side_sign="-1"/>
+  <!-- Depth camera (front & center, same mount as the ToF) -->
+  <xacro:depth_camera/>
   <!-- IMU (gyro + accelerometer), near the body center -->
   <joint name="imu_joint" type="fixed">
